File: DiagramaLogicoFisico.sch (KiCad schematic (older format))
At the start: 5 parts

Commit message: Added subcircuits. Voltage regulator and crystal oscilator
Parts:
- added C? (x2): 22pF, symbol Device:C
- added J?: Conn_01x03, symbol Connector_Generic:Conn_01x03
- added Y?: 20Mhz, symbol Device:Crystal
Connections:
- wire segments 12 -> 27
Changed lines of the file:
@@
 L DSPIC33EP512GM604-I/PT:DSPIC33EP512GM604-I_PT U?
 U 1 1 5E4E75B9
-P 3600 1400
-F 0 "U?" H 8400 1787 60  0000 C CNN
-F 1 "DSPIC33EP512GM604-I_PT" H 8400 1681 60  0000 C CNN
-F 2 "TQFP44_MC" H 8400 1640 60  0001 C CNN
-F 3 "" H 3600 1400 60  0000 C CNN
-	1    3600 1400
+P 3200 2600
+F 0 "U?" H 8000 2987 60  0000 C CNN
+F 1 "DSPIC33EP512GM604-I_PT" H 8000 2881 60  0000 C CNN
+F 2 "TQFP44_MC" H 8000 2840 60  0001 C CNN
+F 3 "" H 3200 2600 60  0000 C CNN
+	1    3200 2600
 	1    0    0    -1
 $EndComp
@@
 	2700 1250 2700 1150
 Connection ~ 2700 1250
+$Comp
+L Connector_Generic:Conn_01x03 J?
+U 1 1 5E54CA6A
+P 2250 2700
+F 0 "J?" H 2330 2742 50  0000 L CNN
+F 1 "Conn_01x03" H 2330 2651 50  0000 L CNN
+F 2 "" H 2250 2700 50  0001 C CNN
+F 3 "~" H 2250 2700 50  0001 C CNN
+	1    2250 2700
+	-1   0    0    1
+$EndComp
+Wire Wire Line
+	3200 2700 2450 2700
+Wire Wire Line
+	3200 2800 2450 2800
+$Comp
+L power:GND #PWR?
+U 1 1 5E554843
+P 2550 2450
+F 0 "#PWR?" H 2550 2200 50  0001 C CNN
+F 1 "GND" H 2555 2277 50  0000 C CNN
+F 2 "" H 2550 2450 50  0001 C CNN
+F 3 "" H 2550 2450 50  0001 C CNN
+	1    2550 2450
+	-1   0    0    1
+$EndComp
+Wire Wire Line
+	2550 2450 2550 2600
+Wire Wire Line
+	2550 2600 2450 2600
+$Comp
+L Device:Crystal Y?
+U 1 1 5E5748B1
+P 1950 5150
+F 0 "Y?" H 1950 5418 50  0000 C CNN
+F 1 "20Mhz" H 1950 5327 50  0000 C CNN
+F 2 "" H 1950 5150 50  0001 C CNN
+F 3 "~" H 1950 5150 50  0001 C CNN
+	1    1950 5150
+	0    1    1    0
+$EndComp
+$Comp
+L Device:C C?
+U 1 1 5E57DCA4
+P 1800 4750
+F 0 "C?" H 1915 4796 50  0000 L CNN
+F 1 "22pF" H 1915 4705 50  0000 L CNN
+F 2 "" H 1838 4600 50  0001 C CNN
+F 3 "~" H 1800 4750 50  0001 C CNN
+	1    1800 4750
+	0    -1   -1   0
+$EndComp
+$Comp
+L power:GND #PWR?
+U 1 1 5E586CC0
+P 900 5650
+F 0 "#PWR?" H 900 5400 50  0001 C CNN
+F 1 "GND" H 905 5477 50  0000 C CNN
+F 2 "" H 900 5650 50  0001 C CNN
+F 3 "" H 900 5650 50  0001 C CNN
+	1    900  5650
+	1    0    0    -1
+$EndComp
+Wire Wire Line
+	1650 4750 900  4750
+Wire Wire Line
+	1650 5600 900  5600
+Connection ~ 900  5600
+Wire Wire Line
+	900  5600 900  5650
+Wire Wire Line
+	1950 5000 1950 4750
+Wire Wire Line
+	900  4700 900  4750
+Wire Wire Line
+	1950 4750 2650 4750
+Wire Wire Line
+	2650 4750 2650 5500
+Wire Wire Line
+	2650 5500 3200 5500
+Connection ~ 1950 4750
+Connection ~ 900  4750
+Wire Wire Line
+	900  4750 900  5600
+Wire Wire Line
+	1950 5300 1950 5600
+Wire Wire Line
+	3200 5600 1950 5600
+$Comp
+L Device:C C?
+U 1 1 5E59F4A1
+P 1800 5600
+F 0 "C?" H 1915 5646 50  0000 L CNN
+F 1 "22pF" H 1915 5555 50  0000 L CNN
+F 2 "" H 1838 5450 50  0001 C CNN
+F 3 "~" H 1800 5600 50  0001 C CNN
+	1    1800 5600
+	0    -1   -1   0
+$EndComp
+Connection ~ 1950 5600
 $EndSCHEMATC

Commit message: Added PWM's, UART's, LED's and Probe conections.
Parts:
- added D? (x3): LED, symbol Device:LED
- added J?: Conn_01x05, symbol Connector_Generic:Conn_01x05
- added J? (x2): Conn_01x03, symbol Connector_Generic:Conn_01x03
- C? (x2): value 30µF -> 1µF
Connections:
- wire segments 27 -> 71
Changed lines of the file:
@@
 P 2700 1600
 F 0 "C?" H 2815 1646 50  0000 L CNN
-F 1 "30µF" H 2815 1555 50  0000 L CNN
+F 1 "1µF" H 2815 1555 50  0000 L CNN
 F 2 "" H 2738 1450 50  0001 C CNN
 F 3 "~" H 2700 1600 50  0001 C CNN
@@
 P 1750 1600
 F 0 "C?" H 1865 1646 50  0000 L CNN
-F 1 "30µF" H 1865 1555 50  0000 L CNN
+F 1 "1µF" H 1865 1555 50  0000 L CNN
 F 2 "" H 1788 1450 50  0001 C CNN
 F 3 "~" H 1750 1600 50  0001 C CNN
@@
 	1950 5000 1950 4750
 Wire Wire Line
-	900  4700 900  4750
-Wire Wire Line
 	1950 4750 2650 4750
 Wire Wire Line
@@
 	2650 5500 3200 5500
 Connection ~ 1950 4750
-Connection ~ 900  4750
 Wire Wire Line
 	900  4750 900  5600
@@
 $EndComp
 Connection ~ 1950 5600
+$Comp
+L Connector_Generic:Conn_01x05 J?
+U 1 1 5E53B068
+P 2200 4400
+F 0 "J?" H 2118 3975 50  0000 C CNN
+F 1 "Conn_01x05" H 2118 4066 50  0000 C CNN
+F 2 "" H 2200 4400 50  0001 C CNN
+F 3 "~" H 2200 4400 50  0001 C CNN
+	1    2200 4400
+	-1   0    0    1
+$EndComp
+Wire Wire Line
+	3200 4900 2750 4900
+Wire Wire Line
+	2750 4900 2750 4600
+Wire Wire Line
+	2750 4600 2400 4600
+Wire Wire Line
+	3200 4800 2800 4800
+Wire Wire Line
+	2800 4800 2800 4500
+Wire Wire Line
+	2800 4500 2400 4500
+Wire Wire Line
+	3200 4300 2800 4300
+Wire Wire Line
+	2800 4300 2800 4400
+Wire Wire Line
+	2800 4400 2400 4400
+$Comp
+L power:GND #PWR?
+U 1 1 5E542BDD
+P 2500 4300
+F 0 "#PWR?" H 2500 4050 50  0001 C CNN
+F 1 "GND" H 2505 4127 50  0000 C CNN
+F 2 "" H 2500 4300 50  0001 C CNN
+F 3 "" H 2500 4300 50  0001 C CNN
+	1    2500 4300
+	0    -1   -1   0
+$EndComp
+$Comp
+L power:+3.3V #PWR?
+U 1 1 5E5477B6
+P 2600 4200
+F 0 "#PWR?" H 2600 4050 50  0001 C CNN
+F 1 "+3.3V" H 2615 4373 50  0000 C CNN
+F 2 "" H 2600 4200 50  0001 C CNN
+F 3 "" H 2600 4200 50  0001 C CNN
+	1    2600 4200
+	0    1    1    0
+$EndComp
+Wire Wire Line
+	2600 4200 2400 4200
+Wire Wire Line
+	2500 4300 2400 4300
+$Comp
+L Connector_Generic:Conn_01x03 J?
+U 1 1 5E55105D
+P 2250 3050
+F 0 "J?" H 2330 3092 50  0000 L CNN
+F 1 "Conn_01x03" H 2330 3001 50  0000 L CNN
+F 2 "" H 2250 3050 50  0001 C CNN
+F 3 "~" H 2250 3050 50  0001 C CNN
+	1    2250 3050
+	-1   0    0    1
+$EndComp
+Wire Wire Line
+	2550 2950 2450 2950
+Wire Wire Line
+	2550 2600 2550 2950
+Connection ~ 2550 2600
+Wire Wire Line
+	3200 2900 2600 2900
+Wire Wire Line
+	2600 2900 2600 3050
+Wire Wire Line
+	2600 3050 2450 3050
+Wire Wire Line
+	3200 3000 2650 3000
+Wire Wire Line
+	2650 3000 2650 3150
+Wire Wire Line
+	2650 3150 2450 3150
+$Comp
+L power:GND #PWR?
+U 1 1 5E55F72C
+P 3050 3100
+F 0 "#PWR?" H 3050 2850 50  0001 C CNN
+F 1 "GND" H 3055 2927 50  0000 C CNN
+F 2 "" H 3050 3100 50  0001 C CNN
+F 3 "" H 3050 3100 50  0001 C CNN
+	1    3050 3100
+	0    1    1    0
+$EndComp
+Wire Wire Line
+	3050 3100 3200 3100
+$Comp
+L power:GND #PWR?
+U 1 1 5E561E34
+P 3050 5400
+F 0 "#PWR?" H 3050 5150 50  0001 C CNN
+F 1 "GND" H 3055 5227 50  0000 C CNN
+F 2 "" H 3050 5400 50  0001 C CNN
+F 3 "" H 3050 5400 50  0001 C CNN
+	1    3050 5400
+	0    1    1    0
+$EndComp
+Wire Wire Line
+	3050 5400 3200 5400
+$Comp
+L power:GND #PWR?
+U 1 1 5E563E98
+P 12950 5200
+F 0 "#PWR?" H 12950 4950 50  0001 C CNN
+F 1 "GND" H 12955 5027 50  0000 C CNN
+F 2 "" H 12950 5200 50  0001 C CNN
+F 3 "" H 12950 5200 50  0001 C CNN
+	1    12950 5200
+	0    -1   -1   0
+$EndComp
+Wire Wire Line
+	12950 5200 12800 5200
+$Comp
+L power:+3.3V #PWR?
+U 1 1 5E56C8F8
+P 3100 5300
+F 0 "#PWR?" H 3100 5150 50  0001 C CNN
+F 1 "+3.3V" H 3115 5473 50  0000 C CNN
+F 2 "" H 3100 5300 50  0001 C CNN
+F 3 "" H 3100 5300 50  0001 C CNN
+	1    3100 5300
+	0    -1   -1   0
+$EndComp
+Wire Wire Line
+	3200 5300 3100 5300
+$Comp
+L Connector_Generic:Conn_01x03 J?
+U 1 1 5E583EF4
+P 2250 3400
+F 0 "J?" H 2330 3442 50  0000 L CNN
+F 1 "Conn_01x03" H 2330 3351 50  0000 L CNN
+F 2 "" H 2250 3400 50  0001 C CNN
+F 3 "~" H 2250 3400 50  0001 C CNN
+	1    2250 3400
+	-1   0    0    1
+$EndComp
+Wire Wire Line
+	3200 4000 2600 4000
+Wire Wire Line
+	2600 4000 2600 3500
+Wire Wire Line
+	2600 3500 2450 3500
+Wire Wire Line
+	3200 3600 2650 3600
+Wire Wire Line
+	2650 3600 2650 3400
+Wire Wire Line
+	2650 3400 2450 3400
+Wire Wire Line
+	3200 3400 2700 3400
+Wire Wire Line
+	2700 3400 2700 3300
+Wire Wire Line
+	2700 3300 2450 3300
+$Comp
+L Device:LED D?
+U 1 1 5E588349
+P 13450 5300
+F 0 "D?" H 13443 5045 50  0000 C CNN
+F 1 "LED" H 13443 5136 50  0000 C CNN
+F 2 "" H 13450 5300 50  0001 C CNN
+F 3 "~" H 13450 5300 50  0001 C CNN
+	1    13450 5300
+	-1   0    0    1
+$EndComp
+$Comp
+L Device:LED D?
+U 1 1 5E591027
+P 13750 5400
+F 0 "D?" H 13743 5145 50  0000 C CNN
+F 1 "LED" H 13743 5236 50  0000 C CNN
+F 2 "" H 13750 5400 50  0001 C CNN
+F 3 "~" H 13750 5400 50  0001 C CNN
+	1    13750 5400
+	-1   0    0    1
+$EndComp
+$Comp
+L Device:LED D?
+U 1 1 5E59369A
+P 14050 5600
+F 0 "D?" H 14043 5345 50  0000 C CNN
+F 1 "LED" H 14043 5436 50  0000 C CNN
+F 2 "" H 14050 5600 50  0001 C CNN
+F 3 "~" H 14050 5600 50  0001 C CNN
+	1    14050 5600
+	-1   0    0    1
+$EndComp
+Wire Wire Line
+	12800 4800 13300 4800
+Wire Wire Line
+	13300 4800 13300 5300
+Wire Wire Line
+	12800 4900 13250 4900
+Wire Wire Line
+	13250 4900 13250 5400
+Wire Wire Line
+	13250 5400 13600 5400
+Wire Wire Line
+	12800 5000 13200 5000
+Wire Wire Line
+	13200 5000 13200 5600
+Wire Wire Line
+	13200 5600 13900 5600
+$Comp
+L power:GND #PWR?
+U 1 1 5E5A4799
+P 14600 5400
+F 0 "#PWR?" H 14600 5150 50  0001 C CNN
+F 1 "GND" H 14605 5227 50  0000 C CNN
+F 2 "" H 14600 5400 50  0001 C CNN
+F 3 "" H 14600 5400 50  0001 C CNN
+	1    14600 5400
+	0    -1   -1   0
+$EndComp
+Wire Wire Line
+	14200 5600 14600 5600
+Wire Wire Line
+	14600 5600 14600 5400
+Wire Wire Line
+	13900 5400 14600 5400
+Connection ~ 14600 5400
+Wire Wire Line
+	13600 5300 14600 5300
+Wire Wire Line
+	14600 5300 14600 5400
 $EndSCHEMATC

Commit message: Added new a new DSP footprint to the diagram
Parts:
- removed C? (x2): 22pF, symbol Device:C
- removed U?: DSPIC33EP512GM604-I_PT, TQFP44_MC, symbol DSPIC33EP512GM604-I/PT:DSPIC33EP512GM604-I_PT
- removed Y?: 20Mhz, symbol Device:Crystal
- added C? (x2): 22pF, symbol Device:C
- added U?: DSPIC33EP128GM604, symbol Norberto:DSPIC33EP128GM604
- added Y?: 7Mhz, symbol Device:Crystal
Connections:
- wire segments 71 -> 85
Other:
- moved on the sheet: D?, J?
