File: DiagramaLogicoFisico.sch (KiCad schematic (older format))
At the start: 49 parts, among them J1 Conn_01x02_Servo1, J10 Conn_01x04_TRIS, J11 Conn_01x04_3v3, J2 Conn_01x03_UART1, J3 Conn_01x03_UART2, J4 Conn_01x04_PWM, J5 Conn_01x05_PROGRAMER, J6 Conn_01x02_POWER, J7 Conn_01x02_Servo2, J8 Conn_01x02_Servo3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

Commit message: Updated Physical diagram
Parts:
- C1: symbol Device:CP1 -> DiagramaLogicoFisico-rescue:CP1-Device
- C10, C2, C3, C4, C5, C6, C7, C8, C9: symbol Device:C -> DiagramaLogicoFisico-rescue:C-Device
- D1, D2, D3: symbol Device:LED -> DiagramaLogicoFisico-rescue:LED-Device
- J1, J6, J7, J8, J9: symbol Connector_Generic:Conn_01x02 -> DiagramaLogicoFisico-rescue:Conn_01x02-Connector_Generic
- J10, J11, J4: symbol Connector_Generic:Conn_01x04 -> DiagramaLogicoFisico-rescue:Conn_01x04-Connector_Generic
- J2, J3: symbol Connector_Generic:Conn_01x03 -> DiagramaLogicoFisico-rescue:Conn_01x03-Connector_Generic
- J5: symbol Connector_Generic:Conn_01x05 -> DiagramaLogicoFisico-rescue:Conn_01x05-Connector_Generic
- R1, R10, R11, R12, R15, R16, R17, R18, R19, R2, R3, R4, R5, R6, R7, R8, R9: symbol Device:R -> DiagramaLogicoFisico-rescue:R-Device
- U1: symbol Regulator_Linear:L7805 -> DiagramaLogicoFisico-rescue:L7805-Regulator_Linear
- U7: symbol Regulator_Linear:AZ1117-3.3 -> DiagramaLogicoFisico-rescue:AZ1117-3.3-Regulator_Linear
- Y1: symbol Device:Crystal -> DiagramaLogicoFisico-rescue:Crystal-Device
Changed lines of the file:
@@
 	19800 11900 19800 11650
 $Comp
-L Device:R R15
+L DiagramaLogicoFisico-rescue:R-Device R15
 U 1 1 5EA0CFA9
 P 19800 11500
@@
 $EndComp
 $Comp
-L Device:R R1
+L DiagramaLogicoFisico-rescue:R-Device R1
 U 1 1 5E722A02
 P 15700 9550
@@
 	14150 11400 14150 11500
 $Comp
-L power:GND #PWR0101
+L DiagramaLogicoFisico-rescue:GND-power #PWR0101
 U 1 1 5E88DDED
 P 14150 11400
@@
 $EndComp
 $Comp
-L Device:CP1 C1
+L DiagramaLogicoFisico-rescue:CP1-Device C1
 U 1 1 5E88CB39
 P 14150 11750
@@
 $EndComp
 $Comp
-L power:+3.3V #PWR0115
+L DiagramaLogicoFisico-rescue:+3.3V-power #PWR0115
 U 1 1 5E7D1F3B
 P 16550 13650
@@
 $EndComp
 $Comp
-L power:GND #PWR0114
+L DiagramaLogicoFisico-rescue:GND-power #PWR0114
 U 1 1 5E7D0D32
 P 16250 13650
@@
 $EndComp
 $Comp
-L power:+3.3V #PWR0113
+L DiagramaLogicoFisico-rescue:+3.3V-power #PWR0113
 U 1 1 5E81BB22
 P 16050 15100
@@
 	16050 15100 16200 15100
 $Comp
-L Device:R R2
+L DiagramaLogicoFisico-rescue:R-Device R2
 U 1 1 5E723556
 P 15900 9550
@@
 $EndComp
 $Comp
-L power:GND #PWR0104
+L DiagramaLogicoFisico-rescue:GND-power #PWR0104
 U 1 1 5E542BDD
 P 16900 16300
@@
 $EndComp
 $Comp
-L power:+3.3V #PWR0105
+L DiagramaLogicoFisico-rescue:+3.3V-power #PWR0105
 U 1 1 5E5477B6
 P 16800 16200
@@
 $EndComp
 $Comp
-L Connector_Generic:Conn_01x05 J5
+L DiagramaLogicoFisico-rescue:Conn_01x05-Connector_Generic J5
 U 1 1 5E53B068
 P 16900 16600
@@
 	16300 13250 16300 13300
 $Comp
-L Device:C C6
+L DiagramaLogicoFisico-rescue:C-Device C6
 U 1 1 5E7DB13D
 P 16400 13450
@@
 	18250 11450 18250 11400
 $Comp
-L Device:C C8
+L DiagramaLogicoFisico-rescue:C-Device C8
 U 1 1 5E7C5DD4
 P 18400 11550
@@
 	16300 10050 16300 10000
 $Comp
-L Device:C C5
+L DiagramaLogicoFisico-rescue:C-Device C5
 U 1 1 5E794CBB
 P 16400 9950
@@
 $EndComp
 $Comp
-L power:+3.3V #PWR0108
+L DiagramaLogicoFisico-rescue:+3.3V-power #PWR0108
 U 1 1 5E60F525
 P 16250 9850
@@
 $EndComp
 $Comp
-L power:GND #PWR0111
+L DiagramaLogicoFisico-rescue:GND-power #PWR0111
 U 1 1 5E62CC50
 P 16550 9850
@@
 	15900 9000 15900 9400
 $Comp
-L Device:R R3
+L DiagramaLogicoFisico-rescue:R-Device R3
 U 1 1 5E725740
 P 16100 9550
@@
 	15150 13900 15150 14300
 $Comp
-L Connector_Generic:Conn_01x04 J4
+L DiagramaLogicoFisico-rescue:Conn_01x04-Connector_Generic J4
 U 1 1 5E6EF778
 P 15250 14500
@@
 	14600 13800 14600 12650
 $Comp
-L power:GND #PWR0112
+L DiagramaLogicoFisico-rescue:GND-power #PWR0112
 U 1 1 5E62F152
 P 18400 11400
@@
 $EndComp
 $Comp
-L power:+3.3V #PWR0109
+L DiagramaLogicoFisico-rescue:+3.3V-power #PWR0109
 U 1 1 5E620108
 P 18400 11700
@@
 	18350 9100 18350 9700
 $Comp
-L Device:Crystal Y1
+L DiagramaLogicoFisico-rescue:Crystal-Device Y1
 U 1 1 5E5BF228
 P 20500 11500
@@
 $EndComp
 $Comp
-L Device:C C4
+L DiagramaLogicoFisico-rescue:C-Device C4
 U 1 1 5E5BF22E
 P 20650 11900
@@
 $EndComp
 $Comp
-L power:GND #PWR0107
+L DiagramaLogicoFisico-rescue:GND-power #PWR0107
 U 1 1 5E5BF234
 P 21550 11000
@@
 	20500 11350 20500 11050
 $Comp
-L Device:C C3
+L DiagramaLogicoFisico-rescue:C-Device C3
 U 1 1 5E5BF246
 P 20650 11050
@@
 	19350 9700 19750 9700
 $Comp
-L power:GND #PWR0106
+L DiagramaLogicoFisico-rescue:GND-power #PWR0106
 U 1 1 5E5A4799
 P 19750 9500
@@
 	18400 9500 18750 9500
 $Comp
-L Device:LED D3
+L DiagramaLogicoFisico-rescue:LED-Device D3
 U 1 1 5E59369A
 P 19200 9700
@@
 $EndComp
 $Comp
-L Device:LED D2
+L DiagramaLogicoFisico-rescue:LED-Device D2
 U 1 1 5E591027
 P 18900 9500
@@
 $EndComp
 $Comp
-L Device:LED D1
+L DiagramaLogicoFisico-rescue:LED-Device D1
 U 1 1 5E588349
 P 18600 9400
@@
 $EndComp
 $Comp
-L Connector_Generic:Conn_01x03 J2
+L DiagramaLogicoFisico-rescue:Conn_01x03-Connector_Generic J2
 U 1 1 5E54CA6A
 P 13350 10650
@@
 $EndComp
 $Comp
-L power:GND #PWR0103
+L DiagramaLogicoFisico-rescue:GND-power #PWR0103
 U 1 1 5E554843
 P 13650 10400
@@
 	13650 10550 13550 10550
 $Comp
-L Connector_Generic:Conn_01x03 J3
+L DiagramaLogicoFisico-rescue:Conn_01x03-Connector_Generic J3
 U 1 1 5E55105D
 P 13350 11000
@@
 	9350 9050 10650 9050
 $Comp
-L Connector_Generic:Conn_01x02 J1
+L DiagramaLogicoFisico-rescue:Conn_01x02-Connector_Generic J1
 U 1 1 5EA81FF7
 P 10850 9150
@@
 Connection ~ 9350 10350
 $Comp
-L Device:R R6
+L DiagramaLogicoFisico-rescue:R-Device R6
 U 1 1 5E802A42
 P 9350 9650
@@
 $EndComp
 $Comp
-L Device:R R5
+L DiagramaLogicoFisico-rescue:R-Device R5
 U 1 1 5E7D6096
 P 9350 9250
@@
 	6250 11650 7050 11650
 $Comp
-L power:+3.3V #PWR0122
+L DiagramaLogicoFisico-rescue:+3.3V-power #PWR0122
 U 1 1 5E906013
 P 10350 14300
@@
 	6250 11550 6450 11550
 $Comp
-L Connector_Generic:Conn_01x02 J6
+L DiagramaLogicoFisico-rescue:Conn_01x02-Connector_Generic J6
 U 1 1 5E83A5B1
 P 6050 11650
@@
 $EndComp
 $Comp
-L power:GND #PWR0119
+L DiagramaLogicoFisico-rescue:GND-power #PWR0119
 U 1 1 5E823902
 P 9350 13900
@@
 $EndComp
 $Comp
-L Device:R R12
+L DiagramaLogicoFisico-rescue:R-Device R12
 U 1 1 5E8238F8
 P 9350 13650
@@
 	9100 13050 9350 13050
 $Comp
-L Device:R R11
+L DiagramaLogicoFisico-rescue:R-Device R11
 U 1 1 5E8238E6
 P 9350 13250
@@
 $EndComp
 $Comp
-L power:GND #PWR0118
+L DiagramaLogicoFisico-rescue:GND-power #PWR0118
 U 1 1 5E8238D1
 P 9350 12600
@@
 $EndComp
 $Comp
-L Device:R R10
+L DiagramaLogicoFisico-rescue:R-Device R10
 U 1 1 5E8238C7
 P 9350 12350
@@
 	9100 11750 9350 11750
 $Comp
-L Device:R R9
+L DiagramaLogicoFisico-rescue:R-Device R9
 U 1 1 5E8238B5
 P 9350 11950
@@
 $EndComp
 $Comp
-L power:GND #PWR0117
+L DiagramaLogicoFisico-rescue:GND-power #PWR0117
 U 1 1 5E81AC95
 P 9350 11200
@@
 $EndComp
 $Comp
-L Device:R R8
+L DiagramaLogicoFisico-rescue:R-Device R8
 U 1 1 5E81AC8B
 P 9350 10950
@@
 	9100 10350 9350 10350
 $Comp
-L Device:R R7
+L DiagramaLogicoFisico-rescue:R-Device R7
 U 1 1 5E81AC79
 P 9350 10550
@@
 	9350 9800 9350 9850
 $Comp
-L power:GND #PWR0116
+L DiagramaLogicoFisico-rescue:GND-power #PWR0116
 U 1 1 5E8034F0
 P 9350 9900
@@
 $EndComp
 $Comp
-L Connector_Generic:Conn_01x02 J7
+L DiagramaLogicoFisico-rescue:Conn_01x02-Connector_Generic J7
 U 1 1 5EB11B49
 P 10850 10450
@@
 $EndComp
 $Comp
-L Connector_Generic:Conn_01x02 J8
+L DiagramaLogicoFisico-rescue:Conn_01x02-Connector_Generic J8
 U 1 1 5EB1E032
 P 10850 11850
@@
 	9650 13150 10650 13150
 $Comp
-L Device:R R4
+L DiagramaLogicoFisico-rescue:R-Device R4
 U 1 1 5E81C5AF
 P 16350 15100
@@
 $EndComp
 $Comp
-L Connector_Generic:Conn_01x02 J9
+L DiagramaLogicoFisico-rescue:Conn_01x02-Connector_Generic J9
 U 1 1 5EB2A570
 P 10850 13150
@@
 Connection ~ 16700 15100
 $Comp
-L Connector_Generic:Conn_01x04 J10
+L DiagramaLogicoFisico-rescue:Conn_01x04-Connector_Generic J10
 U 1 1 5EB8B1CB
 P 17150 14750
@@
 $EndComp
 $Comp
-L power:GND #PWR0102
+L DiagramaLogicoFisico-rescue:GND-power #PWR0102
 U 1 1 5ED1E4A7
 P 18500 13850
@@
 $EndComp
 $Comp
-L Device:R R19
+L DiagramaLogicoFisico-rescue:R-Device R19
 U 1 1 5ED562FD
 P 17900 13500
@@
 	18300 13850 18300 14000
 $Comp
-L Device:R R18
+L DiagramaLogicoFisico-rescue:R-Device R18
 U 1 1 5ED485EB
 P 17900 13750
@@
 $EndComp
 $Comp
-L Device:R R17
+L DiagramaLogicoFisico-rescue:R-Device R17
 U 1 1 5ED3A919
 P 17900 14000
@@
 $EndComp
 $Comp
-L Device:R R16
+L DiagramaLogicoFisico-rescue:R-Device R16
 U 1 1 5ED2CC60
 P 17900 14250
@@
 	17500 14250 17500 13250
 $Comp
-L Connector_Generic:Conn_01x04 J11
+L DiagramaLogicoFisico-rescue:Conn_01x04-Connector_Generic J11
 U 1 1 5F10BC75
 P 11300 14350
@@
 Connection ~ 10900 14250
 $Comp
-L Regulator_Linear:L7805 U1
+L DiagramaLogicoFisico-rescue:L7805-Regulator_Linear U1
 U 1 1 5F1886FD
 P 8150 14300
@@
 $EndComp
 $Comp
-L power:GND #PWR0120
+L DiagramaLogicoFisico-rescue:GND-power #PWR0120
 U 1 1 5E830F1E
 P 8150 15200
@@
 	7050 15100 7650 15100
 $Comp
-L Device:C C2
+L DiagramaLogicoFisico-rescue:C-Device C2
 U 1 1 5F1E9FE0
 P 7650 14500
@@
 	8150 15100 8600 15100
 $Comp
-L Device:C C7
+L DiagramaLogicoFisico-rescue:C-Device C7
 U 1 1 5F24027D
 P 8600 14500
@@
 	8150 15100 8150 15200
 $Comp
-L Regulator_Linear:AZ1117-3.3 U7
+L DiagramaLogicoFisico-rescue:AZ1117-3.3-Regulator_Linear U7
 U 1 1 5F2DEE47
 P 9850 14300
@@
 $EndComp
 $Comp
-L Device:C C9
+L DiagramaLogicoFisico-rescue:C-Device C9
 U 1 1 5F305B75
 P 9050 14500
@@
 Connection ~ 10350 14300
 $Comp
-L Device:C C10
+L DiagramaLogicoFisico-rescue:C-Device C10
 U 1 1 5F41553C
 P 10350 14550
