File: _autosave-DiagramaLogicoFisico.kicad_pcb (KiCad board)
At the start: 2 copper layers, 87.6 x 95.2 mm, 42 parts, among them J1 Conn_01x02_Servo1, J2 Conn_01x03_UART1, J3 Conn_01x03_UART2, J4 Conn_01x04_PWM, J5 Conn_01x05_PROGRAMER, J6 Conn_01x02_POWER, J7 Conn_01x02_Servo2, J8 Conn_01x02_Servo3, J9 Conn_01x02_Servo4, U2 DSPIC33EP128GM604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

Commit message: Proyecto Almost Released Vias
Routing:
- net Net-(J5-Pad5): track 42.4 -> 51.0 mm, vias 0 -> 1
- net Net-(J5-Pad4): track 58.8 -> 64.9 mm, vias 0 -> 1
- net Net-(J3-Pad2): track 64.8 -> 70.4 mm, vias 0 -> 1
- net Net-(J4-Pad1): track 38.9 -> 35.5 mm, vias 0 -> 1
- net Net-(J4-Pad2): track 35.3 -> 32.9 mm, vias 0 -> 1
- net Net-(J4-Pad3): track 33.9 -> 32.1 mm, vias 0 -> 1
- net Net-(J3-Pad1): track 45.5 -> 46.9 mm, vias 0 -> 1
- net Net-(J2-Pad1): track 81.8 -> 82.5 mm, vias 0 -> 1
- net Net-(J4-Pad4): track 33.5 -> 32.8 mm, vias 0 -> 1
- net Net-(J2-Pad2): vias 0 -> 1
