File: DiagramaLogicoFisico.kicad_pcb (KiCad board)
At the start: 2 copper layers, 35 parts, among them J2 Conn_01x03, J3 Conn_01x03, J4 Conn_01x04, J5 Conn_01x05, J6 Conn_01x02, U2 DSPIC33EP128GM604, U3 LM317T/SERVO, U4 LM317T/SERVO, U5 LM317T/SERVO, U6 LM317T/SERVO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

Commit message: Proyecto Almost Released
Parts:
- removed C5TANTALUM1: 10µF, Capacitor_THT:C_Disc_D3.8mm_W2.6mm_P2.50mm
- added C1: Tantalo 10uF, Capacitor_THT:C_Disc_D3.8mm_W2.6mm_P2.50mm, F.Cu at (172.7, 110.5)
- added J1: Conn_01x02_Servo1, TerminalBlock:TerminalBlock_bornier-2_P5.08mm, F.Cu at (152.4, 121.9)
- added J7: Conn_01x02_Servo2, TerminalBlock:TerminalBlock_bornier-2_P5.08mm, F.Cu at (152.4, 104.1)
- added J8: Conn_01x02_Servo3, TerminalBlock:TerminalBlock_bornier-2_P5.08mm, F.Cu at (152.4, 86.4)
- added J9: Conn_01x02_Servo4, TerminalBlock:TerminalBlock_bornier-2_P5.08mm, F.Cu at (152.4, 69.8)
- added R15: 1M, Resistor_THT:R_Axial_DIN0204_L3.6mm_D1.6mm_P5.08mm_Horizontal, F.Cu at (191.8, 97.8)
- J2: value Conn_01x03 -> Conn_01x03_UART1
- J3: value Conn_01x03 -> Conn_01x03_UART2
- J4: value Conn_01x04 -> Conn_01x04_PWM
- J5: value Conn_01x05 -> Conn_01x05_PROGRAMER
- J6: value Conn_01x02 -> Conn_01x02_POWER
- R1, R2, R3: value R -> K2
- Y1: value 7Mhz -> 7.3728Mhz
- moved J5 200.4 mm to (196.8, 142.2), turned to 90 degrees
- moved Y1 174.9 mm to (198.1, 106.7)
- moved R4 171.9 mm to (208.3, 135.9), turned to 180 degrees
- moved J4 170.9 mm to (177.8, 142.2), turned to 90 degrees
- moved U2 168.0 mm to (182.9, 106.7)
- moved J6 159.5 mm to (209.6, 82.5), turned to 90 degrees
- moved R3 156.6 mm to (191.8, 72.4), turned to 270 degrees
- moved J2 147.1 mm to (167.6, 142.2), turned to 270 degrees
- moved U3 146.1 mm to (166.4, 129.5), turned to 180 degrees
- moved R2 144.9 mm to (191.8, 81.3), turned to 270 degrees
- moved R1 144.8 mm to (191.8, 90.2), turned to 270 degrees
- moved R13 141.4 mm to (180.3, 91.4), turned to 90 degrees
- moved U7 141.2 mm to (176.5, 77.5)
- moved J3 139.0 mm to (154.9, 142.2), turned to 270 degrees
- moved C3 137.5 mm to (203.2, 101.6), turned to 90 degrees
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Connections:
- J5 pad 2: Net-(J5-Pad2) -> +3V3
- J5 pad 3: Net-(J5-Pad3) -> GND
- J5 pad 4: GND -> Net-(J5-Pad4)
- J5 pad 5: +3V3 -> Net-(J5-Pad5)
- R11 pad 1: +6V -> Net-(J9-Pad2)
- R4 pad 2: Net-(J5-Pad3) -> Net-(J5-Pad1)
- R5 pad 1: +6V -> Net-(J1-Pad2)
- R7 pad 1: +6V -> Net-(J7-Pad2)
- R9 pad 1: +6V -> Net-(J8-Pad2)
- U2 pad 18: Net-(J5-Pad3) -> Net-(J5-Pad1)
- U2 pad 23: Net-(J5-Pad2) -> Net-(J5-Pad5)
- U2 pad 24: Net-(J5-Pad1) -> Net-(J5-Pad4)
- U3 pad 3: +6V -> Net-(J1-Pad2)
- U4 pad 3: +6V -> Net-(J7-Pad2)
- U5 pad 3: +6V -> Net-(J8-Pad2)
- U6 pad 3: +6V -> Net-(J9-Pad2)
Other:
- board outline added: 87.6 x 95.2 mm
- board text added: "P-ARM-ALMOST"

Commit message: Proyecto Almost Released Vias
Parts:
- added G***: LOGO, Logo:logoUni, F.Cu at (158.8, 62.0)
- added G***: LOGO, Logo:logo2, F.Cu at (202.4, 66.0)
- moved R3 22.9 mm to (191.8, 95.2), turned to 90 degrees
- moved D1 17.8 mm to (200.7, 92.7), turned to 180 degrees
- moved J2 17.8 mm to (149.9, 142.2), turned to 90 degrees
- moved J3 12.9 mm to (167.9, 142.2)
- moved D3 12.8 mm to (200.7, 77.5), turned to 180 degrees
- moved R1 12.7 mm to (191.8, 77.5), turned to 90 degrees
- moved R13 6.84 mm to (182.9, 85.1), turned to 180 degrees
- moved R2 5.08 mm to (191.8, 86.4), turned to 90 degrees
- moved R14 4.58 mm to (177.8, 90.2), turned to 0 degrees
- moved C3 4.58 mm to (207.0, 104.1)
- moved C4 4.58 mm to (201.9, 101.6)
- moved R15 4.58 mm to (195.6, 100.3)
- moved Y1 3.81 mm to (198.1, 110.5)
- moved D2 2.84 mm to (200.7, 85.1), turned to 180 degrees
- moved C5 1.27 mm to (180.3, 96.5)
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Routing:
- net GND: track 0.00 -> 443.9 mm
- net Net-(J6-Pad2): track 0.00 -> 107.9 mm
- net +3V3: track 0.00 -> 105.7 mm
- net Net-(J2-Pad1): track 0.00 -> 81.8 mm
- net Net-(J2-Pad2): track 0.00 -> 75.1 mm
- net Net-(J3-Pad2): track 0.00 -> 64.8 mm
- net Net-(J5-Pad4): track 0.00 -> 58.8 mm
- net Net-(C3-Pad2): track 0.00 -> 47.1 mm
- net Net-(J3-Pad1): track 0.00 -> 45.5 mm
- net Net-(J5-Pad5): track 0.00 -> 42.4 mm
- net Net-(J5-Pad1): track 0.00 -> 41.3 mm
- net Net-(J4-Pad1): track 0.00 -> 38.9 mm
- net Net-(R1-Pad2): track 0.00 -> 36.8 mm
- net Net-(J4-Pad2): track 0.00 -> 35.3 mm
- net Net-(J4-Pad3): track 0.00 -> 33.9 mm
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Other:
- outline, holes or cut-outs redrawn
- board text added: "DSPIC"
- board text added: "P-ARM ALMOST"
- board text added: "POWER"
- board text added: "PROBE"
- board text added: "PWM"
- board text added: "SERVO 1"
- board text added: "SERVO 2"
- board text added: "SERVO 3"
- board text added: "SERVO 4"
- board text added: "TM"
- board text added: "UART1"
- board text added: "UART2"
- board text added: "by NPCMOS"
- board text added: "Δ"
- board text removed: "P-ARM-ALMOST"

Commit message: Proyecto Almost Released Vias
Routing:
- net Net-(J5-Pad5): track 42.4 -> 51.0 mm, vias 0 -> 1
- net Net-(J5-Pad4): track 58.8 -> 64.9 mm, vias 0 -> 1
- net Net-(J3-Pad2): track 64.8 -> 70.4 mm, vias 0 -> 1
- net Net-(J4-Pad1): track 38.9 -> 35.5 mm, vias 0 -> 1
- net Net-(J4-Pad2): track 35.3 -> 32.9 mm, vias 0 -> 1
- net Net-(J4-Pad3): track 33.9 -> 32.1 mm, vias 0 -> 1
- net Net-(J3-Pad1): track 45.5 -> 46.9 mm, vias 0 -> 1
- net Net-(J2-Pad1): track 81.8 -> 82.5 mm, vias 0 -> 1
- net Net-(J4-Pad4): track 33.5 -> 32.8 mm, vias 0 -> 1
- net Net-(J2-Pad2): vias 0 -> 1
