File: PCB_PLANOS_LOGOS_VIAS.kicad_pcb (KiCad board)
At the start: 2 copper layers, 87.6 x 95.2 mm, 42 parts, among them J1 Conn_01x02_Servo1, J2 Conn_01x03_UART1, J3 Conn_01x03_UART2, J4 Conn_01x04_PWM, J5 Conn_01x05_PROGRAMER, J6 Conn_01x02_POWER, J7 Conn_01x02_Servo2, J8 Conn_01x02_Servo3, J9 Conn_01x02_Servo4, U2 DSPIC33EP128GM604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

Commit message: Proyecto Almost Released Vias
Routing:
- net Net-(J5-Pad5): track 42.4 -> 51.0 mm, vias 0 -> 1
- net Net-(J5-Pad4): track 58.8 -> 64.9 mm, vias 0 -> 1
- net Net-(J3-Pad2): track 64.8 -> 70.4 mm, vias 0 -> 1
- net Net-(J4-Pad1): track 38.9 -> 35.5 mm, vias 0 -> 1
- net Net-(J4-Pad2): track 35.3 -> 32.9 mm, vias 0 -> 1
- net Net-(J4-Pad3): track 33.9 -> 32.1 mm, vias 0 -> 1
- net Net-(J3-Pad1): track 45.5 -> 46.9 mm, vias 0 -> 1
- net Net-(J2-Pad1): track 81.8 -> 82.5 mm, vias 0 -> 1
- net Net-(J4-Pad4): track 33.5 -> 32.8 mm, vias 0 -> 1
- net Net-(J2-Pad2): vias 0 -> 1

Commit message: Proyecto Almost Released Vias
Parts:
- moved C5 2.73 mm to (183.1, 96.4)
- renumbered G*** to G****
Routing:
- net Net-(R1-Pad2): track 36.8 -> 41.4 mm
- net GND: track 443.9 -> 447.7 mm
- net Net-(R3-Pad2): track 22.4 -> 19.0 mm
- net +3V3: track 105.7 -> 106.6 mm
- net Net-(R2-Pad2): track 27.6 -> 26.8 mm
Other:
- net class Power added: clearance 0.4, trace_width 0.8, via_dia 0.6, via_drill 0.4
- net class Signal added: clearance 0.3, trace_width 0.4, via_dia 0.4, via_drill 0.3
- rule trace_min: 0.2 -> 0.4

Commit message: Proyecto Almost Released Fixed
Parts:
- removed G****: LOGO, Logo:logo2
- added G***: LOGO, Logo:logo2, F.Cu at (202.7, 67.0)
- moved J4 5.05 mm to (172.8, 142.2)
- moved G*** 4.50 mm to (154.3, 62.3)
- moved J3 2.91 mm to (165.0, 142.2)
- moved J2 2.72 mm to (147.1, 142.2)
Routing:
- net GND: track 447.7 -> 454.2 mm
- net Net-(J4-Pad4): track 32.8 -> 36.4 mm
- net Net-(J3-Pad1): track 46.9 -> 49.6 mm
- net Net-(J2-Pad1): track 82.5 -> 80.8 mm
- net Net-(J3-Pad2): track 70.4 -> 68.8 mm
- net Net-(J4-Pad3): track 32.1 -> 33.1 mm
- net Net-(J2-Pad2): track 75.1 -> 74.5 mm
